File: electronics/esp32-clover/esp32-clover.kicad_pcb (KiCad board)
At the start: 4 copper layers, 29.2 x 46.5 mm, 77 parts, among them J1 USB4055-30-A, J2 BATT_CONN, J3 Conn_01x08_Male, J4 Conn_ARM_JTAG_SWD_10, J5 Conn_01x10_Male, Q1 BC847, SW1 RESET, SW2 BOOT, SW3 PROG_BTN, U1 MCP73832-2-OT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

Commit message: added transfer and stitching vias, closes #1
Routing:
- net GND: track 162.6 -> 159.6 mm, vias 8 -> 67
