File: electronics/esp32-clover/adc.kicad_sch (KiCad schematic)
At the start: 4 parts, among them J6 TBP02R2-381-05BE, U6 ADC124S101CIMM

Commit message: update before switching to stm32
Parts:
- J6: footprint CUI_TBP02R2-381-05BE -> TBP02R2-381-05BE:CUI_TBP02R2-381-05BE
- U6: footprint SOP50P490X110-10N -> ADC124S101CIMM:ADC124S101CIMM
Connections:
- net GPIO4/ADC_CS renamed ADC_CS
Other:
- note added: "TODO Replace PART"
Changed lines of the file:
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@@
     (stroke (width 0) (type default))
   )
+  (text "TODO Replace PART" (at 113.03 120.65 0)
+    (effects (font (size 4 4)) (justify left bottom))
+  )
   (label "ADC_IN4" (at 158.115 99.695 0) (fields_autoplaced)
     (effects (font (size 1.27 1.27)) (justify left bottom))
@@
     (effects (font (size 1.27 1.27)) (justify right))
   )
-  (hierarchical_label "GPIO4{slash}ADC_CS" (shape input) (at 116.205 94.615 180) (fields_autoplaced)
+  (hierarchical_label "ADC_CS" (shape input) (at 116.205 94.615 180) (fields_autoplaced)
     (effects (font (size 1.27 1.27)) (justify right))
   )
@@
         )
         (path "/845f0d6a-9016-490e-9296-0668f78ddd1b/f09230ab-00b9-4398-8896-254b056bb6a1"
-          (reference "C?") (unit 1)
+          (reference "C9") (unit 1)
         )
       )
@@
         )
         (path "/845f0d6a-9016-490e-9296-0668f78ddd1b/f09230ab-00b9-4398-8896-254b056bb6a1"
-          (reference "#PWR077") (unit 1)
+          (reference "#PWR044") (unit 1)
         )
       )
@@
         )
         (path "/845f0d6a-9016-490e-9296-0668f78ddd1b/f09230ab-00b9-4398-8896-254b056bb6a1"
-          (reference "#PWR090") (unit 1)
+          (reference "#PWR047") (unit 1)
         )
       )
@@
         )
         (path "/845f0d6a-9016-490e-9296-0668f78ddd1b/f09230ab-00b9-4398-8896-254b056bb6a1"
-          (reference "#PWR089") (unit 1)
+          (reference "#PWR046") (unit 1)
         )
       )
@@
         )
         (path "/845f0d6a-9016-490e-9296-0668f78ddd1b/f09230ab-00b9-4398-8896-254b056bb6a1"
-          (reference "#PWR076") (unit 1)
+          (reference "#PWR048") (unit 1)
         )
       )
@@
         )
         (path "/845f0d6a-9016-490e-9296-0668f78ddd1b/f09230ab-00b9-4398-8896-254b056bb6a1"
-          (reference "#PWR088") (unit 1)
+          (reference "#PWR045") (unit 1)
         )
       )
@@
         )
         (path "/845f0d6a-9016-490e-9296-0668f78ddd1b/f09230ab-00b9-4398-8896-254b056bb6a1"
-          (reference "C?") (unit 1)
+          (reference "C8") (unit 1)
         )
       )
@@
       (effects (font (size 1.27 1.27)))
     )
-    (property "Footprint" "SOP50P490X110-10N" (at 128.27 95.885 0)
+    (property "Footprint" "ADC124S101CIMM:ADC124S101CIMM" (at 128.27 95.885 0)
       (effects (font (size 1.27 1.27)) (justify bottom) hide)
     )
@@
         )
         (path "/845f0d6a-9016-490e-9296-0668f78ddd1b/f09230ab-00b9-4398-8896-254b056bb6a1"
-          (reference "U?") (unit 1)
+          (reference "U5") (unit 1)
         )
       )
@@
       (effects (font (size 1.27 1.27)) (justify left) hide)
     )
-    (property "Footprint" "CUI_TBP02R2-381-05BE" (at 191.135 97.155 0)
+    (property "Footprint" "TBP02R2-381-05BE:CUI_TBP02R2-381-05BE" (at 191.135 97.155 0)
       (effects (font (size 1.27 1.27)) (justify bottom) hide)
     )
@@
         )
         (path "/845f0d6a-9016-490e-9296-0668f78ddd1b/f09230ab-00b9-4398-8896-254b056bb6a1"
-          (reference "J?") (unit 1)
-        )
-      )
+          (reference "J7") (unit 1)
+        )
+      )
