File: electronics/esp32-clover/can.kicad_sch (KiCad schematic)
At the start: 10 parts

Commit message: update before switching to stm32
Parts:
- removed J?: TBP02R2-381-05BE, CUI_TBP02R2-381-05BE, symbol TBP02R2-381-05BE:TBP02R2-381-05BE
- added J?: TBP02R2-381-05BE, connectors:TBP02R2-381-05BE, symbol connectors:TBP02R2-381-05BE
- S?: footprint SW_DS01-254-S-01BE -> DS01-254-S-01BE:SW_DS01-254-S-01BE
- gave numbers to parts that had none: 1
Connections:
- net +5V: now also J?.1
- net CAN_H: now also J?.2
- net CAN_INT: now also J?.4
- net CAN_L: now also J?.3
- net GND: now also J?.5
Other:
- note added: "CAN Controller"
- note added: "CAN Transceiver"
- note added: "Connector"
- note added: "Level Shifting"
- note added: "Selectable Termination"
- moved on the sheet: C?, R?, S?, U2, Y?
