File: electronics/esp32-clover/dac.kicad_sch (KiCad schematic)
At the start: 5 parts, among them J7 TBP02R2-381-05BE, U8 MCP4728

Commit message: update before switching to stm32
Parts:
- removed J7: TBP02R2-381-05BE, CUI_TBP02R2-381-05BE, symbol TBP02R2-381-05BE:TBP02R2-381-05BE
- added J?: TBP02R2-381-05BE, connectors:TBP02R2-381-05BE, symbol connectors:TBP02R2-381-05BE
Connections:
- net DAC_VOUTA: now also J?.1
- net DAC_VOUTB: now also J?.2
- net DAC_VOUTC: now also J?.3
- net DAC_VOUTD: now also J?.4
- net GND: now also J?.5
- net ADC_LDAC renamed DAC_LDAC
- net ADC_RDY/BSY renamed DAC_RDY/BSY
Changed lines of the file:
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@@
     (effects (font (size 1.27 1.27)) (justify right))
   )
-  (hierarchical_label "ADC_LDAC" (shape input) (at 129.54 113.03 180) (fields_autoplaced)
+  (hierarchical_label "DAC_LDAC" (shape input) (at 129.54 113.03 180) (fields_autoplaced)
     (effects (font (size 1.27 1.27)) (justify right))
   )
@@
     (effects (font (size 1.27 1.27)) (justify right))
   )
-  (hierarchical_label "ADC_RDY{slash}BSY" (shape output) (at 102.87 115.57 180) (fields_autoplaced)
+  (hierarchical_label "DAC_RDY{slash}BSY" (shape output) (at 102.87 115.57 180) (fields_autoplaced)
     (effects (font (size 1.27 1.27)) (justify right))
   )
@@
         )
         (path "/845f0d6a-9016-490e-9296-0668f78ddd1b/4ce35da5-c24d-4786-9252-9aee302acd2a"
-          (reference "#PWR069") (unit 1)
+          (reference "#PWR062") (unit 1)
         )
       )
@@
         )
         (path "/845f0d6a-9016-490e-9296-0668f78ddd1b/4ce35da5-c24d-4786-9252-9aee302acd2a"
-          (reference "C?") (unit 1)
+          (reference "C10") (unit 1)
         )
       )
@@
         )
         (path "/845f0d6a-9016-490e-9296-0668f78ddd1b/4ce35da5-c24d-4786-9252-9aee302acd2a"
-          (reference "#PWR043") (unit 1)
+          (reference "#PWR060") (unit 1)
         )
       )
@@
         )
         (path "/845f0d6a-9016-490e-9296-0668f78ddd1b/4ce35da5-c24d-4786-9252-9aee302acd2a"
-          (reference "#PWR091") (unit 1)
+          (reference "#PWR063") (unit 1)
         )
       )
@@
         )
         (path "/845f0d6a-9016-490e-9296-0668f78ddd1b/4ce35da5-c24d-4786-9252-9aee302acd2a"
-          (reference "C?") (unit 1)
-        )
-      )
-    )
-  )
-  (symbol (lib_id "power:+3.3V") (at 107.95 107.95 0) (unit 1)
-    (in_bom yes) (on_board yes) (dnp no) (fields_autoplaced)
-    (property "Reference" "#PWR068" (at 107.95 111.76 0)
-      (effects (font (size 1.27 1.27)) hide)
-    )
-    (property "Value" "+3.3V" (at 107.95 104.3742 0)
-      (effects (font (size 1.27 1.27)))
-    )
-    (property "Footprint" "" (at 107.95 107.95 0)
-      (effects (font (size 1.27 1.27)) hide)
-    )
-    (property "Datasheet" "" (at 107.95 107.95 0)
-      (effects (font (size 1.27 1.27)) hide)
-    )
-    (pin "1")
-    (instances
-      (project "esp32-clover"
-        (path "/845f0d6a-9016-490e-9296-0668f78ddd1b"
-          (reference "#PWR068") (unit 1)
-        )
-        (path "/845f0d6a-9016-490e-9296-0668f78ddd1b/4ce35da5-c24d-4786-9252-9aee302acd2a"
-          (reference "#PWR035") (unit 1)
-        )
-      )
-    )
-  )
-  (symbol (lib_id "TBP02R2-381-05BE:TBP02R2-381-05BE") (at 183.515 113.03 0) (unit 1)
-    (in_bom yes) (on_board yes) (dnp no)
-    (property "Reference" "J7" (at 182.245 103.505 0)
-      (effects (font (size 1.27 1.27)) (justify left))
-    )
-    (property "Value" "TBP02R2-381-05BE" (at 190.5 114.935 0)
-      (effects (font (size 1.27 1.27)) (justify left) hide)
-    )
-    (property "Footprint" "CUI_TBP02R2-381-05BE" (at 183.515 113.03 0)
+          (reference "C11") (unit 1)
+        )
+      )
+    )
+  )
+  (symbol (lib_id "connectors:TBP02R2-381-05BE") (at 183.515 113.03 0) (unit 1)
+    (in_bom yes) (on_board yes) (dnp no) (fields_autoplaced)
+    (property "Reference" "J?" (at 189.865 111.76 0)
+      (effects (font (size 1.27 1.27)) (justify left))
+    )
+    (property "Value" "TBP02R2-381-05BE" (at 189.865 114.3 0)
+      (effects (font (size 1.27 1.27)) (justify left))
+    )
+    (property "Footprint" "connectors:TBP02R2-381-05BE" (at 183.515 113.03 0)
       (effects (font (size 1.27 1.27)) (justify bottom) hide)
     )
@@
       (project "esp32-clover"
         (path "/845f0d6a-9016-490e-9296-0668f78ddd1b"
-          (reference "J7") (unit 1)
-        )
-        (path "/845f0d6a-9016-490e-9296-0668f78ddd1b/4ce35da5-c24d-4786-9252-9aee302acd2a"
           (reference "J?") (unit 1)
         )
+        (path "/845f0d6a-9016-490e-9296-0668f78ddd1b/5369a936-2211-41e4-96f5-8eaefadf9c59"
+          (reference "J?") (unit 1)
+        )
+        (path "/845f0d6a-9016-490e-9296-0668f78ddd1b/4ce35da5-c24d-4786-9252-9aee302acd2a"
+          (reference "J?") (unit 1)
+        )
+      )
+    )
+  )
+  (symbol (lib_id "power:+3.3V") (at 107.95 107.95 0) (unit 1)
+    (in_bom yes) (on_board yes) (dnp no) (fields_autoplaced)
+    (property "Reference" "#PWR068" (at 107.95 111.76 0)
+      (effects (font (size 1.27 1.27)) hide)
+    )
+    (property "Value" "+3.3V" (at 107.95 104.3742 0)
+      (effects (font (size 1.27 1.27)))
+    )
+    (property "Footprint" "" (at 107.95 107.95 0)
+      (effects (font (size 1.27 1.27)) hide)
+    )
+    (property "Datasheet" "" (at 107.95 107.95 0)
+      (effects (font (size 1.27 1.27)) hide)
+    )
+    (pin "1")
+    (instances
+      (project "esp32-clover"
+        (path "/845f0d6a-9016-490e-9296-0668f78ddd1b"
+          (reference "#PWR068") (unit 1)
+        )
+        (path "/845f0d6a-9016-490e-9296-0668f78ddd1b/4ce35da5-c24d-4786-9252-9aee302acd2a"
+          (reference "#PWR058") (unit 1)
+        )
       )
     )
@@
         )
         (path "/845f0d6a-9016-490e-9296-0668f78ddd1b/4ce35da5-c24d-4786-9252-9aee302acd2a"
-          (reference "#PWR045") (unit 1)
+          (reference "#PWR061") (unit 1)
         )
       )
@@
         )
         (path "/845f0d6a-9016-490e-9296-0668f78ddd1b/4ce35da5-c24d-4786-9252-9aee302acd2a"
-          (reference "#PWR042") (unit 1)
+          (reference "#PWR059") (unit 1)
         )
       )
@@
         )
         (path "/845f0d6a-9016-490e-9296-0668f78ddd1b/4ce35da5-c24d-4786-9252-9aee302acd2a"
-          (reference "U?") (unit 1)
+          (reference "U8") (unit 1)
         )
       )
@@
         )
         (path "/845f0d6a-9016-490e-9296-0668f78ddd1b/4ce35da5-c24d-4786-9252-9aee302acd2a"
-          (reference "R?") (unit 1)
-        )
-      )
+          (reference "R14") (unit 1)
+        )
+      )
