File: electronics/esp32-clover/gpio.kicad_sch (KiCad schematic)
At the start: 4 parts, among them U5 TCA9534

Commit message: update before switching to stm32
Parts:
- added J? (x2): TBP02R2-381-05BE, connectors:TBP02R2-381-05BE, symbol connectors:TBP02R2-381-05BE
- added R11: 4.7K, Resistor_SMD:R_0603_1608Metric, symbol Device:R
- added U5: TCA9534, Package_SO:TSSOP-16_4.4x5mm_P0.65mm, symbol Interface_Expansion:TCA9534
Connections:
- net +3.3V: now also R11.2, U5.1 (A0), U5.16 (VDD)
- net GND: now also J?.3, J?.4, J?.5, U5.2 (A1), U5.3 (A2), U5.8 (GND)
- net I2C_SCL: now also U5.14 (SCL)
- net I2C_SDA: now also U5.15 (SDA)
- net GPIO1_P7 renamed GPIO1_P7/PV_RST
- new net GPIO2_INT: R11.1, U5.13 (~{INT})
- new net GPIO2_P1: J?.1, U5.5 (P1)
- new net GPIO2_P1/DAC_LDAC: U5.4 (P0)
- new net GPIO2_P2: J?.2, U5.6 (P2)
- new net GPIO2_P3: J?.3, U5.7 (P3)
- new net GPIO2_P4: J?.4, U5.9 (P4)
- new net GPIO2_P5: J?.5, U5.10 (P5)
- new net GPIO2_P6: J?.1, U5.11 (P6)
- new net GPIO2_P7: J?.2, U5.12 (P7)
Other:
- note added: "Address: 0x21"
- note added: "Status"
- moved on the sheet: D5, R11, R16, U5
