File: electronics/esp32-clover/sd.kicad_sch (KiCad schematic)
At the start: 3 parts

Commit message: update before switching to stm32
Parts:
- removed J?: ST1W008S4AR1500, JAE_ST1W008S4AR1500, symbol ST1W008S4AR1500:ST1W008S4AR1500
- added J?: ST1W008S4AR1500, card_connectors:ST1W008S4AR1500, symbol card_connectors:ST1W008S4AR1500
- gave numbers to parts that had none: 2
Connections:
- net +3.3V: now also J?.4 (VCC)
- net GND: now also J?.GND1 (GND), J?.GND2 (GND), J?.GND3 (GND), J?.GND4 (GND)
- net SD_CS: now also J?.2 (CS)
- net SPI_MISO: now also J?.7 (MISO)
- net SPI_MOSI: now also J?.3 (MOSI)
- net SPI_SCK: now also J?.5 (SCK)
- net at Q4.3 (D): now also J?.6 (GND)
Changed lines of the file:
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@@
   (symbol (lib_id "Transistor_FET:BSS214NW") (at 132.715 104.775 0) (unit 1)
     (in_bom yes) (on_board yes) (dnp no) (fields_autoplaced)
-    (property "Reference" "Q?" (at 138.43 104.14 0)
+    (property "Reference" "Q4" (at 138.43 104.14 0)
       (effects (font (size 1.27 1.27)) (justify left))
     )
@@
       (project "esp32-clover"
         (path "/845f0d6a-9016-490e-9296-0668f78ddd1b/7df621dc-9aa9-4ef0-97a0-5baf9e162604"
-          (reference "Q?") (unit 1)
+          (reference "Q4") (unit 1)
         )
       )
@@
   (symbol (lib_id "Device:R") (at 118.745 104.775 90) (unit 1)
     (in_bom yes) (on_board yes) (dnp no) (fields_autoplaced)
-    (property "Reference" "R?" (at 118.745 100.33 90)
+    (property "Reference" "R39" (at 118.745 100.33 90)
       (effects (font (size 1.27 1.27)))
     )
@@
       (project "esp32-clover"
         (path "/845f0d6a-9016-490e-9296-0668f78ddd1b/7df621dc-9aa9-4ef0-97a0-5baf9e162604"
-          (reference "R?") (unit 1)
+          (reference "R39") (unit 1)
         )
       )
@@
   (symbol (lib_id "power:GND") (at 153.035 103.505 0) (unit 1)
     (in_bom yes) (on_board yes) (dnp no) (fields_autoplaced)
-    (property "Reference" "#PWR03" (at 153.035 109.855 0)
+    (property "Reference" "#PWR0111" (at 153.035 109.855 0)
       (effects (font (size 1.27 1.27)) hide)
     )
@@
       (project "esp32-clover"
         (path "/845f0d6a-9016-490e-9296-0668f78ddd1b/7df621dc-9aa9-4ef0-97a0-5baf9e162604"
-          (reference "#PWR03") (unit 1)
+          (reference "#PWR0111") (unit 1)
         )
       )
@@
   (symbol (lib_id "power:+3.3V") (at 153.035 88.265 90) (unit 1)
     (in_bom yes) (on_board yes) (dnp no)
-    (property "Reference" "#PWR02" (at 156.845 88.265 0)
+    (property "Reference" "#PWR0110" (at 156.845 88.265 0)
       (effects (font (size 1.27 1.27)) hide)
     )
@@
       (project "esp32-clover"
         (path "/845f0d6a-9016-490e-9296-0668f78ddd1b/7df621dc-9aa9-4ef0-97a0-5baf9e162604"
-          (reference "#PWR02") (unit 1)
+          (reference "#PWR0110") (unit 1)
         )
       )
@@
   (symbol (lib_id "power:GND") (at 135.255 109.855 0) (unit 1)
     (in_bom yes) (on_board yes) (dnp no) (fields_autoplaced)
-    (property "Reference" "#PWR010" (at 135.255 116.205 0)
+    (property "Reference" "#PWR0109" (at 135.255 116.205 0)
       (effects (font (size 1.27 1.27)) hide)
     )
@@
       (project "esp32-clover"
         (path "/845f0d6a-9016-490e-9296-0668f78ddd1b/7df621dc-9aa9-4ef0-97a0-5baf9e162604"
-          (reference "#PWR010") (unit 1)
+          (reference "#PWR0109") (unit 1)
         )
       )
     )
   )
-  (symbol (lib_id "ST1W008S4AR1500:ST1W008S4AR1500") (at 163.195 90.805 0) (unit 1)
+  (symbol (lib_id "card_connectors:ST1W008S4AR1500") (at 163.195 90.805 0) (unit 1)
     (in_bom yes) (on_board yes) (dnp no) (fields_autoplaced)
-    (property "Reference" "J?" (at 169.545 91.44 0)
+    (property "Reference" "J?" (at 169.545 90.805 0)
       (effects (font (size 1.27 1.27)) (justify left))
     )
-    (property "Value" "ST1W008S4AR1500" (at 169.545 93.98 0)
+    (property "Value" "ST1W008S4AR1500" (at 169.545 93.345 0)
       (effects (font (size 1.27 1.27)) (justify left))
     )
-    (property "Footprint" "JAE_ST1W008S4AR1500" (at 163.195 90.805 0)
+    (property "Footprint" "card_connectors:ST1W008S4AR1500" (at 163.195 90.805 0)
       (effects (font (size 1.27 1.27)) (justify bottom) hide)
     )
@@
       (effects (font (size 1.27 1.27)) (justify bottom) hide)
     )
+    (pin "GND1")
+    (pin "GND2")
+    (pin "GND3")
+    (pin "GND4")
     (pin "1")
     (pin "2")
@@
     (pin "7")
     (pin "8")
-    (pin "GND1")
-    (pin "GND2")
-    (pin "GND3")
-    (pin "GND4")
     (instances
       (project "esp32-clover"
